Commit message: fill()
Fill all todos

File: urdf/robot.xacro (robot description, xacro)
@@ -23,6 +23,4 @@
   <xacro:property name="Iz_wheel" value="${0.5 * wheel_mass * wheel_link_radius * wheel_link_radius}"/>
   <xacro:property name="I_wheel" value="${(1.0/12.0) * wheel_mass * (3.0 * wheel_link_radius * wheel_link_radius + wheel_link_length * wheel_link_length)}"/>
-  <!-- Gazebo definitions -->
-  <xacro:include filename="$(find robot_model_pkg)/urdf/robot.gazebo"/>
   <!-- Dummy link -->
   <link name="dummy"/>
@@ -34,4 +32,5 @@
       </geometry>
       <origin rpy="0 0 0" xyz="0 0 0"/>
+      <material name="Red"/>
     </visual>
     <collision>
@@ -52,5 +51,4 @@
     </inertial>
   </link>
-  <!-- Fixed joint between dummy and body -->
   <joint name="dummy_joint" type="fixed">
     <parent link="dummy"/>
@@ -61,14 +59,28 @@
     <link name="${name}">
       <visual>
-        <!-- TODO: Complete -->
+        <geometry>
+          <cylinder radius="${wheel_link_radius}" length="${wheel_link_length}"/>
+        </geometry>
+        <origin xyz="0 0 0" rpy="1.5708 0 0"/>
+        <material name="Black"/>
       </visual>
       <collision>
-        <!-- TODO: Complete -->
+        <geometry>
+          <cylinder radius="${wheel_link_radius}" length="${wheel_link_length}"/>
+        </geometry>
+        <origin xyz="0 0 0" rpy="1.5708 0 0"/>
       </collision>
       <inertial>
-        <!-- TODO: Complete -->
+        <mass value="${wheel_mass}"/>
+        <inertia ixx="${I_wheel}" ixy="0" ixz="0"
+                 iyy="${I_wheel}" iyz="0"
+                 izz="${Iz_wheel}"/>
+      </inertial>
     </link>
     <joint name="${name}_joint" type="${joint_type}">
-      <!-- TODO: Complete -->
+      <parent link="body_link"/>
+      <child link="${name}"/>
+      <origin xyz="${x} ${y} ${z}" rpy="0 0 0"/>
+      <axis xyz="0 1 0"/>
       <limit effort="1000" velocity="1000"/>
       <dynamics damping="1.0" friction="1.0"/>
@@ -76,11 +88,14 @@
   </xacro:macro>
   <!-- Instantiate wheels -->
-  <xacro:wheel name="rear_right_wheel"  x="${-body_link_x_dim/2 + 1.2*wheel_link_radius}" y="${-body_link_y_dim/2 - 1.2*wheel_link_length/2}" z="${wheel_link_z_location}" joint_type="continuous"/>
-  <!-- TODO: Complete: Wheels must be named - rear_left_wheel, front_right_wheel, front_left_wheel -->
-<!-- Camera -->
+  <xacro:wheel name="rear_right_wheel"  x="${-body_link_x_dim/2 + 0.2}" y="${-body_link_y_dim/2 - 0.05}" z="${wheel_link_z_location}" joint_type="continuous"/>
+  <xacro:wheel name="rear_left_wheel"   x="${-body_link_x_dim/2 + 0.2}" y="${ body_link_y_dim/2 + 0.05}" z="${wheel_link_z_location}" joint_type="continuous"/>
+  <xacro:wheel name="front_right_wheel" x="${ body_link_x_dim/2 - 0.2}" y="${-body_link_y_dim/2 - 0.05}" z="${wheel_link_z_location}" joint_type="continuous"/>
+  <xacro:wheel name="front_left_wheel"  x="${ body_link_x_dim/2 - 0.2}" y="${ body_link_y_dim/2 + 0.05}" z="${wheel_link_z_location}" joint_type="continuous"/>
+  <!-- Camera -->
   <link name="camera_link">
     <visual>
       <geometry><box size="${sensor_side} ${sensor_side} ${sensor_side}"/></geometry>
       <origin rpy="0 0 0" xyz="0 0 0" />
+      <material name="Green"/>
     </visual>
     <collision>
@@ -105,15 +120,39 @@
   <!-- Sonar -->
   <link name="sonar_link">
-    <!-- TODO: Complete -->
+    <visual>
+      <geometry>
+        <cylinder radius="0.02" length="0.05"/>
+      </geometry>
+      <origin rpy="0 0 0" xyz="0 0 0"/>
+      <material name="Blue"/>
+    </visual>
+    <inertial>
+      <mass value="${sensor_mass}"/>
+      <inertia ixx="1e-6" ixy="0" ixz="0" iyy="1e-6" iyz="0" izz="1e-6"/>
+    </inertial>
   </link>
   <joint name="sonar_joint" type="fixed">
-    <!-- TODO: Complete -->
+    <parent link="body_link"/>
+    <child link="sonar_link"/>
+    <origin xyz="0.3 0 ${body_link_z_dim/2}"/>
   </joint>
   <!-- Lidar -->
   <link name="lidar_link">
-    <!-- TODO: Complete -->
+    <visual>
+      <geometry>
+        <cylinder radius="0.05" length="0.02"/>
+      </geometry>
+      <origin rpy="0 0 0" xyz="0 0 0"/>
+      <material name="White"/>
+    </visual>
+    <inertial>
+      <mass value="${sensor_mass}"/>
+      <inertia ixx="1e-6" ixy="0" ixz="0" iyy="1e-6" iyz="0" izz="1e-6"/>
+    </inertial>
   </link>
   <joint name="lidar_joint" type="fixed">
-    <!-- TODO: Complete -->
+    <parent link="body_link"/>
+    <child link="lidar_link"/>
+    <origin xyz="0 0 ${body_link_z_dim/2 + 0.05}"/>
   </joint>
 </robot>
